Commit message: update

File: ROS2_HUMBLE/src/stararm102_description/urdf/stararm102_description.urdf (robot description, URDF)
Before this commit: robot stararm102_description, 10 links, 9 joints
Joints:
- joint joint7_left: limit lower=0 upper=0.025 effort=5 velocity=3.14 -> lower=-1.57 upper=1.57 effort=5 velocity=3.14; type prismatic -> revolute
- joint joint7_right: limit lower=-0.025 upper=0 effort=5 velocity=3.14 -> lower=-1.57 upper=1.57 effort=5 velocity=3.14; mimic joint=joint7_left -> joint=joint7_left multiplier=-1; type prismatic -> revolute

File: ROS2_HUMBLE/src/stararm102_gazebo/urdf/gazebo_configs.urdf.xacro (robot description, xacro)
@@ -92,4 +92,9 @@
             <state_interface name="velocity"/>
         </joint>
+        <joint name="joint7_right">
+            <command_interface name="position"/>
+            <param name="mimic">joint7_left</param>
+            <param name="multiplier">-1</param>
+        </joint>
     </ros2_control>
     <gazebo>

File: ROS2_HUMBLE/src/stararm102_gazebo/urdf/stararm102_gazebo.urdf (robot description, URDF)
Before this commit: robot stararm102_description, 9 links, 8 joints
Joints:
- joint joint7_left: limit lower=0 upper=0.025 effort=1 velocity=3.14 -> lower=-1.57 upper=1.57 effort=1 velocity=3.14; type prismatic -> revolute
- joint joint7_right: limit lower=-0.025 upper=0 effort=1 velocity=3.14 -> lower=-1.57 upper=1.57 effort=1 velocity=3.14; mimic joint=joint7_left -> joint=joint7_left multiplier=-1; type prismatic -> revolute

Commit message: update urdf

File: ROS2_HUMBLE/src/stararm102_description/urdf/stararm102_description.urdf (robot description, URDF)
Before this commit: robot stararm102_description, 10 links, 9 joints
Links:
- link link1: mass 0.0490447462840961 -> 0.0490447462840962
- link link2: mass 0.0902416570859392 -> 0.0902416560384624
- link link3: mass 0.092247950009267 -> 0.0922479500092671
- link link5: mass 0.0455712723510246 -> 0.0455712723510248
Joints:
- joint joint1: origin xyz=0 0 0.04475 rpy=0 0 0 -> xyz=0 0 0.0447500000000019 rpy=0 0 0
- joint joint2: origin xyz=0.02775 0 0.061925 rpy=1.5708 -1.5708 0 -> xyz=0.0277499999999987 0 0.0619249999999976 rpy=1.5707963267949 -1.5707963267949 0
- joint joint3: origin xyz=0.11225 -0.026175 0 rpy=0 0 -1.5708 -> xyz=0.112250000000003 -0.026175000000001 0 rpy=0 0 -1.5707963267949
- joint joint4: origin xyz=0.14117 0 0 rpy=0 0 0 -> xyz=0.141174999999997 0 0 rpy=0 0 0
- joint joint5: origin xyz=0.029 0 0 rpy=-1.5708 0 0 -> xyz=0.0290000000000017 0 0 rpy=-1.5707963267949 0 0
- joint joint7_left: limit lower=-1.57 upper=1.57 effort=5 velocity=3.14 -> lower=-1.57 upper=0 effort=5 velocity=3.14; origin xyz=0 0.00090027 0 rpy=1.5708 0 -1.5708 -> xyz=-0.0123250000000028 0.00010027139309185 -0.071129999999999 rpy=1.5707963267949 -1.5707963267949 0
- joint joint7_right: limit lower=-1.57 upper=1.57 effort=5 velocity=3.14 -> lower=-1.57 upper=0 effort=5 velocity=3.14; origin xyz=0 0.00090027 0 rpy=1.5708 0 -1.5708 -> xyz=0.009675 0.00010027 -0.07113 rpy=1.5708 -1.5708 0

File: ROS2_HUMBLE/src/stararm102_gazebo/urdf/stararm102_gazebo.urdf (robot description, URDF)
Before this commit: robot stararm102_description, 9 links, 8 joints
Links:
- link link1: mass 0.0490447462840961 -> 0.0490447462840962
- link link2: mass 0.0902416570859392 -> 0.0902416560384624
- link link3: mass 0.092247950009267 -> 0.0922479500092671
- link link5: mass 0.0455712723510246 -> 0.0455712723510248
Joints:
- joint joint1: origin xyz=0 0 0.04475 rpy=0 0 0 -> xyz=0 0 0.0447500000000019 rpy=0 0 0
- joint joint2: origin xyz=0.02775 0 0.061925 rpy=1.5708 -1.5708 0 -> xyz=0.0277499999999987 0 0.0619249999999976 rpy=1.5707963267949 -1.5707963267949 0
- joint joint3: origin xyz=0.11225 -0.026175 0 rpy=0 0 -1.5708 -> xyz=0.112250000000003 -0.026175000000001 0 rpy=0 0 -1.5707963267949
- joint joint4: origin xyz=0.14117 0 0 rpy=0 0 0 -> xyz=0.141174999999997 0 0 rpy=0 0 0
- joint joint5: origin xyz=0.029 0 0 rpy=-1.5708 0 0 -> xyz=0.0290000000000017 0 0 rpy=-1.5707963267949 0 0
- joint joint7_left: origin xyz=0 0.00090027 0 rpy=1.5708 0 -1.5708 -> xyz=-0.0123250000000028 0.00010027139309185 -0.071129999999999 rpy=1.5707963267949 -1.5707963267949 0
- joint joint7_right: origin xyz=0 0.00090027 0 rpy=1.5708 0 -1.5708 -> xyz=0.009675 0.00010027 -0.07113 rpy=1.5708 -1.5708 0

Commit message: update

File: ROS2_HUMBLE/src/stararm102_description/urdf/stararm102_description.urdf (robot description, URDF)
Before this commit: robot stararm102_description, 10 links, 9 joints
Joints:
- joint joint7_left: limit lower=-1.57 upper=0 effort=5 velocity=3.14 -> lower=0 upper=1.57 effort=5 velocity=3.14
- joint joint7_right: axis 0 0 -1 -> 0 0 1; limit lower=-1.57 upper=0 effort=5 velocity=3.14 -> lower=0 upper=1.57 effort=5 velocity=3.14

File: ROS2_HUMBLE/src/stararm102_gazebo/urdf/stararm102_gazebo.urdf (robot description, URDF)
Before this commit: robot stararm102_description, 9 links, 8 joints
Joints:
- joint joint7_left: limit lower=-1.57 upper=1.57 effort=1 velocity=3.14 -> lower=0 upper=1.57 effort=1 velocity=3.14
- joint joint7_right: axis 0 0 -1 -> 0 0 1; limit lower=-1.57 upper=1.57 effort=1 velocity=3.14 -> lower=0 upper=1.57 effort=1 velocity=3.14

Commit message: update normal

File: ROS2_HUMBLE/src/stararm102_description/urdf/stararm102_description.urdf (robot description, URDF)
Before this commit: robot stararm102_description, 10 links, 9 joints
Joints:
- joint joint7_right: limit lower=0 upper=1.57 effort=5 velocity=3.14 -> lower=-1.57 upper=0 effort=5 velocity=3.14

File: ROS2_HUMBLE/src/stararm102_gazebo/urdf/gazebo_configs.urdf.xacro (robot description, xacro)
@@ -94,4 +94,8 @@
         <joint name="joint7_right">
             <command_interface name="position"/>
+            <state_interface name="position">
+                <param name="initial_value">0</param>
+            </state_interface>
+            <state_interface name="velocity"/>
             <param name="mimic">joint7_left</param>
             <param name="multiplier">-1</param>

File: ROS2_HUMBLE/src/stararm102_gazebo/urdf/stararm102_gazebo.urdf (robot description, URDF)
Before this commit: robot stararm102_description, 9 links, 8 joints
Joints:
- joint joint7_right: limit lower=0 upper=1.57 effort=1 velocity=3.14 -> lower=-1.57 upper=0 effort=1 velocity=3.14

File: ROS2_HUMBLE/src/stararm102_moveit_config/config/stararm102_description.ros2_control.xacro (robot description, xacro)
@@ -56,9 +56,19 @@
       <command_interface name="position">
         <param name="min">0</param>
-        <param name="max">0.025</param>
+        <param name="max">1.57</param>
       </command_interface>
       <state_interface name="position"/>
       <state_interface name="velocity"/>
     </joint>
+    <joint name="joint7_right">
+      <command_interface name="position">
+        <param name="min">-1.57</param>
+        <param name="max">0</param>
+      </command_interface>
+      <state_interface name="position"/>
+      <state_interface name="velocity"/>
+      <param name="mimic">joint7_left</param>
+      <param name="multiplier">-1</param>
+    </joint>
   </ros2_control>
 </robot>

Commit message: update: 更新新的模型

File: ROS2_HUMBLE/src/stararm102_description/urdf/stararm102_description.urdf (robot description, URDF)
Before this commit: robot stararm102_description, 10 links, 9 joints
Links:
- link base_link: mass 0.133140629988521 -> 0.155441639095221
- link link1: mass 0.0490447462840962 -> 0.0365919096309897
- link link2: mass 0.0902416560384624 -> 0.0677741447743621
- link link3: mass 0.0922479500092671 -> 0.062483417986533
- link link4: mass 0.0298155768600067 -> 0.0290020616470162
- link link5: mass 0.0455712723510248 -> 0.04381347428302
- link link6: mass 0.0277279216939168 -> 0.0277279215984807
- link link7_left: mass 0.0255901502803906 -> 0.0209012827567763
- link link7_right: mass 0.0246485351672712 -> 0.019895
Joints:
- joint joint1: origin xyz=0 0 0.0447500000000019 rpy=0 0 0 -> xyz=0 0 0.0283500000000012 rpy=0 0 0
- joint joint2: limit lower=-1.57 upper=1.57 effort=100 velocity=1 -> lower=0 upper=3.14 effort=100 velocity=1; origin xyz=0.0277499999999987 0 0.0619249999999976 rpy=1.5707963267949 -1.5707963267949 0 -> xyz=0.000100000000001007 0 0.0620250000000017 rpy=-1.5707963267949 0 3.14159265358979
- joint joint3: limit lower=-1.57 upper=1.57 effort=100 velocity=1 -> lower=-3.14 upper=0 effort=100 velocity=1; origin xyz=0.112250000000003 -0.026175000000001 0 rpy=0 0 -1.5707963267949 -> xyz=0.120565306190578 -0.0100999999999999 0.0259999999999978 rpy=0 0 -1.5707963267949
- joint joint4: limit lower=-1.57 upper=1.57 effort=100 velocity=1 -> lower=-1.57 upper=2.2 effort=100 velocity=1; origin xyz=0.141174999999997 0 0 rpy=0 0 0 -> xyz=0.0162194771204603 -0.107604056191361 -0.0259999999999976 rpy=0 0 -1.5707963267949
- joint joint5: limit lower=-1.57 upper=1.57 effort=100 velocity=1 -> lower=-1.2 upper=1.2 effort=100 velocity=1; origin xyz=0.0290000000000017 0 0 rpy=-1.5707963267949 0 0 -> xyz=0.0350000000000005 -0.0013799999999997 0 rpy=-1.57079632679489 0 0
- joint joint6: limit lower=-2.27 upper=2.27 effort=100 velocity=1 -> lower=-3.14 upper=3.14 effort=100 velocity=1; origin xyz=0.14968 0 0.0038453 rpy=-1.5708 0 -1.5708 -> xyz=0.15168 0 0.005225 rpy=-1.5708 0 -1.5708
- joint joint7_left: axis 0 0 1 -> 0 0 -1; origin xyz=-0.0123250000000028 0.00010027139309185 -0.071129999999999 rpy=1.5707963267949 -1.5707963267949 0 -> xyz=0.012325 0 -0.07313 rpy=1.5708 -1.5708 0
- joint joint7_right: axis 0 0 1 -> 0 0 -1; origin xyz=0.009675 0.00010027 -0.07113 rpy=1.5708 -1.5708 0 -> xyz=-0.009675 0 -0.07313 rpy=1.5708 -1.5708 0

File: ROS2_HUMBLE/src/stararm102_gazebo/urdf/stararm102_gazebo.urdf (robot description, URDF)
Before this commit: robot stararm102_description, 9 links, 8 joints
Links:
- link base_link: mass 0.133140629988521 -> 0.155441639095221
- link link1: mass 0.0490447462840962 -> 0.0365919096309897
- link link2: mass 0.0902416560384624 -> 0.0677741447743621
- link link3: mass 0.0922479500092671 -> 0.062483417986533
- link link4: mass 0.0298155768600067 -> 0.0290020616470162
- link link5: mass 0.0455712723510248 -> 0.04381347428302
- link link6: mass 0.0277279216939168 -> 0.0277279215984807
- link link7_left: mass 0.0255901502803906 -> 0.0209012827567763
- link link7_right: mass 0.0246485351672712 -> 0.019895
Joints:
- joint joint1: limit lower=-2.27 upper=2.27 effort=1 velocity=1 -> lower=-2.27 upper=2.27 effort=100 velocity=1; origin xyz=0 0 0.0447500000000019 rpy=0 0 0 -> xyz=0 0 0.0283500000000012 rpy=0 0 0
- joint joint2: limit lower=-1.57 upper=1.57 effort=2.3 velocity=1 -> lower=0 upper=3.14 effort=100 velocity=1; origin xyz=0.0277499999999987 0 0.0619249999999976 rpy=1.5707963267949 -1.5707963267949 0 -> xyz=0.000100000000001007 0 0.0620250000000017 rpy=-1.5707963267949 0 3.14159265358979
- joint joint3: limit lower=-1.57 upper=1.57 effort=2.3 velocity=1 -> lower=-3.14 upper=0 effort=100 velocity=1; origin xyz=0.112250000000003 -0.026175000000001 0 rpy=0 0 -1.5707963267949 -> xyz=0.120565306190578 -0.0100999999999999 0.0259999999999978 rpy=0 0 -1.5707963267949
- joint joint4: limit lower=-1.57 upper=1.57 effort=1 velocity=1 -> lower=-1.57 upper=2.2 effort=100 velocity=1; origin xyz=0.141174999999997 0 0 rpy=0 0 0 -> xyz=0.0162194771204603 -0.107604056191361 -0.0259999999999976 rpy=0 0 -1.5707963267949
- joint joint5: limit lower=-1.57 upper=1.57 effort=1 velocity=1 -> lower=-1.2 upper=1.2 effort=100 velocity=1; origin xyz=0.0290000000000017 0 0 rpy=-1.5707963267949 0 0 -> xyz=0.0350000000000005 -0.0013799999999997 0 rpy=-1.57079632679489 0 0
- joint joint6: limit lower=-2.27 upper=2.27 effort=1 velocity=1 -> lower=-3.14 upper=3.14 effort=100 velocity=1; origin xyz=0.14968 0 0.0038453 rpy=-1.5708 0 -1.5708 -> xyz=0.15168 0 0.005225 rpy=-1.5708 0 -1.5708
- joint joint7_left: axis 0 0 1 -> 0 0 -1; limit lower=0 upper=1.57 effort=1 velocity=3.14 -> lower=0 upper=1.57 effort=5 velocity=3.14; origin xyz=-0.0123250000000028 0.00010027139309185 -0.071129999999999 rpy=1.5707963267949 -1.5707963267949 0 -> xyz=0.012325 0 -0.07313 rpy=1.5708 -1.5708 0
- joint joint7_right: axis 0 0 1 -> 0 0 -1; limit lower=-1.57 upper=0 effort=1 velocity=3.14 -> lower=-1.57 upper=0 effort=5 velocity=3.14; origin xyz=0.009675 0.00010027 -0.07113 rpy=1.5708 -1.5708 0 -> xyz=-0.009675 0 -0.07313 rpy=1.5708 -1.5708 0
